Commit message: first commit

File: src/Lite3_Model_Control/high_level_sim/src/robot_description/lite3_description/xacro/body.xacro (robot description, xacro)
@@ -1,4 +1,6 @@
 <?xml version="1.0"?>
 <robot xmlns:xacro="http://www.ros.org/wiki/xacro">
+    <xacro:property name="M_PI" value="3.1415926535897931" />
+    <xacro:macro name="Lite3" params="has_lidar:=false lidar_hz:=10 lidar_horizontal_samples:=3600 lidar_channels:=16 lidar_min_range:=0.3 lidar_max_range:=130.0 lidar_noise:=0.008">
     <xacro:include filename="$(find lite3_description)/xacro/imu_link.xacro"/>
     <link name="TORSO">
@@ -391,3 +393,100 @@
       <child link="HR_FOOT" />
     </joint>
+    <!-- Lidar -->
+      <xacro:if value="${has_lidar}">
+        <joint name="lidar_base_mount_joint" type="fixed">
+          <origin xyz="0.1745 0 0.05"/>
+          <parent link="TORSO"/>
+          <child link="lidar_base_link"/>
+        </joint>
+        <link name="lidar_base_link">
+          <inertial>
+            <mass value="1e-7"/>
+            <origin xyz="0 0 0.03585"/>
+            <inertia ixx="1e-7" ixy="0" ixz="0" iyy="1e-7" iyz="0" izz="1e-7"/>
+          </inertial>
+          <visual>
+            <geometry>
+              <mesh filename="package://velodyne_description/meshes/VLP16_base_1.dae" />
+            </geometry>
+          </visual>
+          <visual>
+            <geometry>
+              <mesh filename="package://velodyne_description/meshes/VLP16_base_2.dae" />
+            </geometry>
+          </visual>
+          <collision>
+            <origin rpy="0 0 0" xyz="0 0 0.03585"/>
+            <geometry>
+              <cylinder radius="0.0516" length="0.0717"/>
+            </geometry>
+          </collision>
+        </link>
+        <joint name="lidar_base_scan_joint" type="fixed" >
+          <origin xyz="0 0 0.0377" rpy="0 0 0" />
+          <parent link="lidar_base_link" />
+          <child link="lidar_link"/>
+        </joint>
+        <link name="lidar_link">
+          <inertial>
+            <mass value="1e-7"/>
+            <origin xyz="0 0 0"/>
+            <inertia ixx="1e-7" ixy="0" ixz="0" iyy="1e-7" iyz="0" izz="1e-7"/>
+          </inertial>
+          <visual>
+            <origin xyz="0 0 -0.0377" />
+            <geometry>
+              <mesh filename="package://velodyne_description/meshes/VLP16_scan.dae" />
+            </geometry>
+          </visual>
+          <collision>
+            <geometry>
+              <sphere radius="0"/>
+            </geometry>
+          </collision>
+        </link>
+        <gazebo reference="lidar_link">
+          <sensor type="gpu_ray" name="velodyne-VLP16">
+            <pose>0 0 0 0 0 0</pose>
+            <visualize>false</visualize>
+            <update_rate>${lidar_hz}</update_rate>
+            <ray>
+              <scan>
+                <horizontal>
+                  <samples>${lidar_horizontal_samples}</samples>
+                  <resolution>1</resolution>
+                  <min_angle>-${M_PI}</min_angle>
+                  <max_angle>${M_PI}</max_angle>
+                </horizontal>
+                <vertical>
+                  <samples>${lidar_channels}</samples>
+                  <resolution>1</resolution>
+                  <min_angle>-${15.0*M_PI/180.0}</min_angle>
+                  <max_angle> ${15.0*M_PI/180.0}</max_angle>
+                </vertical>
+              </scan>
+              <range>
+                <min>0.3</min>
+                <max>${lidar_max_range+1}</max>
+                <resolution>0.001</resolution>
+              </range>
+              <noise>
+                <type>gaussian</type>
+                <mean>0.0</mean>
+                <stddev>0.0</stddev>
+              </noise>
+            </ray>
+            <plugin name="gazebo_ros_laser_controller" filename="libgazebo_ros_velodyne_gpu_laser.so">
+              <robotNamespace>lite3_gazebo</robotNamespace>
+              <topicName>point_cloud</topicName>
+              <frameName>/lidar_link</frameName>
+              <organize_cloud>false</organize_cloud>
+              <min_range>${lidar_min_range}</min_range>
+              <max_range>${lidar_max_range}</max_range>
+              <gaussianNoise>${lidar_noise}</gaussianNoise>
+            </plugin>
+          </sensor>
+        </gazebo>
+      </xacro:if>
+    </xacro:macro>
 </robot>

File: src/Lite3_Model_Control/high_level_sim/src/robot_description/lite3_description/xacro/robot_with_lidar.xacro (robot description, xacro)
@@ -4,4 +4,13 @@
     <xacro:include filename="$(find lite3_description)/xacro/body.xacro"/>
     <xacro:include filename="$(find lite3_description)/xacro/transmission.xacro"/>
-    <xacro:Lite3 has_lidar="false"/>
+    <!-- Lidar parameters -->
+    <xacro:Lite3
+        has_lidar="true"
+        lidar_hz="20"
+        lidar_horizontal_samples="3600"
+        lidar_channels="16"
+        lidar_min_range="0.3"
+        lidar_max_range="130.0"
+        lidar_noise="0.008"
+    />
 </robot>
